File: pcb/VISP-PCB/VISP-I2C-DUAL/sensors.sch (EAGLE design)
At the start: 47 parts, among them IC1 BMP388, IC2 BMP388, IC3 BMP388, IC4 BMP388, Q1 BSS138, Q2 BSS138, Q3 BSS138, Q4 BSS138, U1 MIC5225-3.3, U3 24C01ASM, U5 BMP280, U6 BMP280, U7 BMP280, U8 BMP280

Commit message: JLCPCB Proven - Dual I2C board with BMP280/SLP06-007 footprints
Parts:
- removed C10, C11, C12, C8: 100nF, Capacitor:CAPACITOR-1206
- removed IC1, IC2, IC3, IC4: BMP388, microbuilder:BMP388
- added GOLD_ORB_SM1: OSHWLOGOLOGO8MM, oshw:OSHWLOGOLOGO8MM
- C1, C3: device microbuilder:CAP_CERAMIC0603_NO -> microbuilder:CAP_CERAMIC_0805
- C9: device Capacitor:CAPACITOR-0603 -> Capacitor:CAPACITOR-0402
- R1, R2, R3, R5, R6, R7, R8, R9: device microbuilder:RESISTOR0805_NOOUTLINE -> microbuilder:RESISTOR_0402
- R4: value 47 Ohm -> 47R; device Resistor:RESISTOR-0603 -> Resistor:RESISTOR-0402
Connections:
- net 3.3V: no longer C10.C1, C11.C1, C12.C1, C8.C1, IC1.CSB, IC1.VDD, IC1.VDDIO, IC2.CSB, IC2.SDO, IC2.VDD, IC2.VDDIO, IC3.CSB, IC3.VDD, IC3.VDDIO, IC4.CSB, IC4.SDO, IC4.VDD, IC4.VDDIO
- net GND: no longer C10.C2, C11.C2, C12.C2, C8.C2, IC1.GND, IC1.SDO, IC2.GND, IC3.GND, IC3.SDO, IC4.GND
- net SCK1_3V: no longer IC3.SCK, IC4.SCK
- net SCK2_3V: no longer IC1.SCK, IC2.SCK
- net SDI1_3V: no longer IC3.SDI, IC4.SDI
- net SDI2_3V: no longer IC1.SDI, IC2.SDI
Other:
- note removed: "Alternate 1206 Bypass Caps (U5->U8)"
