File: pcb/VISP-PCB/VISP-I2C-MUX/sensors.brd (EAGLE design)
At the start: 20.2 x 39.9 mm, 41 parts, among them IC1 BMP388, IC2 BMP388, IC3 BMP388, IC4 BMP388, U1 MIC5225-3.3, U2 TCA9546APWR, U3 24C01ASM, U5 BMP280, U6 BMP280, U7 BMP280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

Commit message: Add BME680 footprints.   Rearrange sensors on the buses to match each other. Bus1 is 2 sensors in same hole, all BMP388's are I2C:0x76 and BME680's are I2C:0x77
Parts:
- U5, U6, U7, U8: value BMP280 -> BME280; device bosch-bmp280:BMP280 -> microbuilder:BME280
- moved IC3 8.00 mm to (14.0, 5.50)
- moved IC4 8.00 mm to (14.0, 13.5)
- moved U5 0.35 mm to (13.8, 2.75), turned to 270 degrees
- moved U6 0.35 mm to (13.8, 10.8), turned to 270 degrees
- moved U7 0.35 mm to (5.75, 10.8), turned to 270 degrees
- moved U8 0.35 mm to (5.75, 2.75), turned to 270 degrees
Connections:
- net 3.3V: now also U5.5, U7.5; no longer IC2.5, IC4.5
- net GND: now also IC2.5, IC4.5; no longer U5.5, U7.5
- net SCK1_3V: now also IC3.2; no longer U6.4
- net SCK2_3V: now also IC4.2, U6.4; no longer U7.4, U8.4
- net SCK3_3V: now also IC1.2, U7.4; no longer IC3.2, IC4.2
- net SCK4_3V: now also U8.4; no longer IC1.2
- net SDI1_3V: now also IC3.4; no longer U6.3
- net SDI2_3V: now also IC4.4, U6.3; no longer U7.3, U8.3
- net SDI3_3V: now also IC1.4, U7.3; no longer IC3.4, IC4.4
- net SDI4_3V: now also U8.3; no longer IC1.4
Routing:
- net GND: track 128.0 -> 174.8 mm, vias 0 -> 11
- net A1: track 19.4 -> 58.5 mm
- net SCK4_3V: track 36.9 -> 73.4 mm, vias 3 -> 4
- net A2: track 31.6 -> 53.1 mm, vias 4 -> 3
- net SDA_5V: track 43.5 -> 22.7 mm
- net A0: track 14.5 -> 30.3 mm, vias 2 -> 3
- net SCK3_3V: track 37.5 -> 51.1 mm
- net SDI4_3V: track 35.1 -> 48.5 mm, vias 3 -> 5
- net SCK2_3V: track 38.9 -> 27.7 mm, vias 2 -> 3
- net SCL_5V: track 26.0 -> 36.4 mm, vias 1 -> 0
- net 3.3V: track 128.1 -> 136.5 mm, vias 2 -> 7
- net SDI2_3V: track 31.2 -> 22.9 mm
- net SCK1_3V: track 39.8 -> 35.3 mm
- net RESET: track 7.65 -> 3.75 mm
- net SDI3_3V: track 32.8 -> 29.0 mm, vias 3 -> 4
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Other:
- board text added: "V0.3"
- board text removed: "V0.2"
